Commit message: write a camera.xacro file.

File: mec_mobile_description/urdf/robots/robot_3d.urdf.xacro (robot description, xacro)
@@ -1,35 +1,58 @@
-<?xml version="1.0"?>
-<robot name="robot_3d" xmlns:xacro="http://www.ros.org/wiki/xacro" xmlns:gz="http://gazebosim.org/schema">
+<?xml version="1.0" ?>
+<robot
+    name="robot_3d"
+    xmlns:xacro="http://www.ros.org/wiki/xacro"
+    xmlns:gz="http://gazebosim.org/schema"
+>
     <xacro:property name="M_PI" value="3.1415926535897931" />
-    <xacro:arg name="robot_name" default="robot_3d"/>
-    <xacro:arg name="prefix" default=""/>
-    <xacro:arg name="use_gazebo" default="false"/>
-    <xacro:include filename="$(find mec_mobile_description)/urdf/mech/robot_3d_base.urdf.xacro"/>
-    <xacro:include filename="$(find mec_mobile_description)/urdf/mech/mecanum_wheel.urdf.xacro"/>
-    <xacro:include filename="$(find mec_mobile_description)/urdf/sensors/rgbd_camera.urdf.xacro"/>
-    <xacro:include filename="$(find mec_mobile_description)/urdf/sensors/lidar.urdf.xacro"/>
-    <xacro:include filename="$(find mec_mobile_description)/urdf/sensors/imu.urdf.xacro"/>
-    <xacro:include filename="$(find mec_mobile_description)/urdf/control/mec_mobile.gazebo"/>
-    <xacro:robot_3d_base prefix="$(arg prefix)"/>
+    <xacro:arg name="robot_name" default="robot_3d" />
+    <xacro:arg name="prefix" default="" />
+    <xacro:arg name="use_gazebo" default="false" />
+    <xacro:include
+        filename="$(find mec_mobile_description)/urdf/mech/robot_3d_base.urdf.xacro"
+    />
+    <xacro:include
+        filename="$(find mec_mobile_description)/urdf/mech/mecanum_wheel.urdf.xacro"
+    />
+    <!-- <xacro:include
+        filename="$(find mec_mobile_description)/urdf/sensors/rgbd_camera.urdf.xacro"
+    /> -->
+    <xacro:include
+        filename="$(find mec_mobile_description)/urdf/sensors/lidar.urdf.xacro"
+    />
+    <xacro:include
+        filename="$(find mec_mobile_description)/urdf/sensors/imu.urdf.xacro"
+    />
+    <xacro:include
+        filename="$(find mec_mobile_description)/urdf/control/mec_mobile.gazebo"
+    />
+    <xacro:include
+        filename="$(find mec_mobile_description)/urdf/sensors/camera.xacro"
+    />
+    <xacro:robot_3d_base prefix="$(arg prefix)" />
     <xacro:mecanum_wheel
-      prefix="$(arg prefix)"
-      side="front_left"
-      x_reflect="1"
-      y_reflect="1"/>
+        prefix="$(arg prefix)"
+        side="front_left"
+        x_reflect="1"
+        y_reflect="1"
+    />
     <xacro:mecanum_wheel
-      prefix="$(arg prefix)"
-      side="front_right"
-      x_reflect="1"
-      y_reflect="-1"/>
+        prefix="$(arg prefix)"
+        side="front_right"
+        x_reflect="1"
+        y_reflect="-1"
+    />
     <xacro:mecanum_wheel
-      prefix="$(arg prefix)"
-      side="back_left"
-      x_reflect="-1"
-      y_reflect="1"/>
+        prefix="$(arg prefix)"
+        side="back_left"
+        x_reflect="-1"
+        y_reflect="1"
+    />
     <xacro:mecanum_wheel
-      prefix="$(arg prefix)"
-      side="back_right"
-      x_reflect="-1"
-      y_reflect="-1"/>
+        prefix="$(arg prefix)"
+        side="back_right"
+        x_reflect="-1"
+        y_reflect="-1"
+    />
     <!-- <xacro:rgbd_camera
       prefix="$(arg prefix)"
@@ -38,20 +61,22 @@
       rpy_offset="0 0 0"/> -->
     <xacro:lidar_sensor
-      prefix="$(arg prefix)"
-      parent="base_link"
-      frame_id="laser_frame"
-      xyz_offset="0 0 0.0825"
-      rpy_offset="0 0 3.14"
-      mesh_xyz_offset="0 0 0"
-      mesh_rpy_offset="${-M_PI/2} 0 0"
-      topic_name="scan"/>
+        prefix="$(arg prefix)"
+        parent="base_link"
+        frame_id="laser_frame"
+        xyz_offset="0 0 0.0825"
+        rpy_offset="0 0 3.14"
+        mesh_xyz_offset="0 0 0"
+        mesh_rpy_offset="${-M_PI/2} 0 0"
+        topic_name="scan"
+    />
     <xacro:imu_sensor
-      prefix="$(arg prefix)"
-      parent="base_link"
-      frame_id="imu"
-      xyz_offset="0 0 0.006"
-      rpy_offset="0 0 0"
-      update_rate="15.0"
-      topic_name="imu/data"/>
+        prefix="$(arg prefix)"
+        parent="base_link"
+        frame_id="imu"
+        xyz_offset="0 0 0.006"
+        rpy_offset="0 0 0"
+        update_rate="15.0"
+        topic_name="imu/data"
+    />
     <!-- 2.4 add Gazebo frictions -->
     <gazebo reference='front_left_wheel_link'>
@@ -114,7 +139,7 @@
     <!-- 2.5.1 Camera physical properties -->
     <joint type="fixed" name="camera_joint">
-      <origin xyz="0.092 0 0.05" rpy="0 0 0"/>
-      <child link="camera_link"/>
-      <parent link="base_link"/>
+      <origin xyz="0.092 0 0.05" rpy="0 0 0" />
+      <child link="camera_link" />
+      <parent link="base_link" />
       <axis xyz="0 1 0" />
     </joint>
@@ -122,21 +147,18 @@
       <pose>0 0 0 0 0 0</pose>
       <inertial>
-        <mass value="0.1"/>
-        <origin xyz="0 0 0" rpy="0 0 0"/>
-        <inertia
-            ixx="1e-6" ixy="0" ixz="0"
-            iyy="1e-6" iyz="0"
-            izz="1e-6"/>
+        <mass value="0.1" />
+        <origin xyz="0 0 0" rpy="0 0 0" />
+        <inertia ixx="1e-6" ixy="0" ixz="0" iyy="1e-6" iyz="0" izz="1e-6" />
       </inertial>
       <collision name='collision'>
-        <origin xyz="0 0 0" rpy="0 0 0"/>
+        <origin xyz="0 0 0" rpy="0 0 0" />
         <geometry>
-          <box size=".03 .03 .03"/>
+          <box size=".03 .03 .03" />
         </geometry>
       </collision>
       <visual name='camera_link_visual'>
-        <origin xyz="0 0 0" rpy="0 0 0"/>
+        <origin xyz="0 0 0" rpy="0 0 0" />
         <geometry>
-          <box size=".02 .02 .02"/>
+          <box size=".02 .02 .02" />
         </geometry>
       </visual>
@@ -146,7 +168,7 @@
     </gazebo>
     <joint type="fixed" name="camera_optical_joint">
-      <origin xyz="0 0 0" rpy="-1.5707 0 -1.5707"/>
-      <child link="camera_link_optical"/>
-      <parent link="camera_link"/>
+      <origin xyz="0 0 0" rpy="-1.5707 0 -1.5707" />
+      <child link="camera_link_optical" />
+      <parent link="camera_link" />
     </joint>
     <link name="camera_link_optical">

Commit message: fix camera. TODO: fix arena.dae file

File: mec_mobile_description/urdf/robots/robot_3d.urdf.xacro (robot description, xacro)
@@ -27,7 +27,7 @@
         filename="$(find mec_mobile_description)/urdf/control/mec_mobile.gazebo"
     />
-    <xacro:include
+    <!-- <xacro:include
         filename="$(find mec_mobile_description)/urdf/sensors/camera.xacro"
-    />
+    /> -->
     <xacro:robot_3d_base prefix="$(arg prefix)" />
     <xacro:mecanum_wheel
@@ -174,4 +174,28 @@
     <link name="camera_link_optical">
     </link>
+    <gazebo reference="camera_link_optical">
+      <sensor type="camera" name="cam_1">
+        <update_rate>30.0</update_rate>
+        <camera>
+          <horizontal_fov>1.047</horizontal_fov>
+          <image>
+            <width>640</width>
+            <height>480</height>
+            <format>R8G8B8</format>
+          </image>
+          <clip>
+            <near>0.1</near>
+            <far>100</far>
+          </clip>
+        </camera>
+        <plugin name="camera_controller" filename="libgazebo_ros_camera.so">
+          <alwaysOn>true</alwaysOn>
+          <updateRate>30.0</updateRate>
+          <cameraName>cam_1</cameraName>
+          <imageTopicName>camera/image_raw</imageTopicName>
+          <frameName>camera_link_optical</frameName>
+        </plugin>
+      </sensor>
+    </gazebo>
     <!-- 2.5.1 End -->
 </robot>

File: mec_mobile_description/urdf/sensors/camera.xacro (robot description, xacro)
@@ -1,23 +1,23 @@
-<?xml version="1.0"?>
-<robot xmlns:xacro="http://www.ros.org/wiki/xacro" >
+<?xml version="1.0" ?>
+<robot xmlns:xacro="http://www.ros.org/wiki/xacro">
     <joint name="camera_joint" type="fixed">
-        <parent link="chassis"/>
-        <child link="camera_link"/>
-        <origin xyz="0.305 0 0.08" rpy="0 0 0"/>
+        <parent link="base_link" />
+        <child link="camera_link" />
+        <origin xyz="0.305 0 0.08" rpy="0 0 0" />
     </joint>
     <link name="camera_link">
         <visual>
             <geometry>
-                <box size="0.010 0.03 0.03"/>
+                <box size="0.010 0.03 0.03" />
             </geometry>
-            <material name="red"/>
+            <material name="red" />
         </visual>
     </link>
     <joint name="camera_optical_joint" type="fixed">
-        <parent link="camera_link"/>
-        <child link="camera_link_optical"/>
-        <origin xyz="0 0 0" rpy="${-pi/2} 0 ${-pi/2}"/>
+        <parent link="camera_link" />
+        <child link="camera_link_optical" />
+        <origin xyz="0 0 0" rpy="${-pi/2} 0 ${-pi/2}" />
     </joint>
-    <link name="camera_link_optical"></link>
+    <link name="camera_link_optical" />
     <gazebo reference="camera_link">
         <material>Gazebo/Red</material>

Commit message: remove build files.

File: mec_mobile_description/urdf/robots/robot_3d.urdf.xacro (robot description, xacro)
@@ -139,5 +139,5 @@
     <!-- 2.5.1 Camera physical properties -->
     <joint type="fixed" name="camera_joint">
-      <origin xyz="0.092 0 0.05" rpy="0 0 0" />
+      <origin xyz="0.092 0 0.05" rpy="-1.57 0 0" />
       <child link="camera_link" />
       <parent link="base_link" />

Commit message: fix camera positioning.

File: mec_mobile_description/urdf/robots/robot_3d.urdf.xacro (robot description, xacro)
@@ -139,5 +139,5 @@
     <!-- 2.5.1 Camera physical properties -->
     <joint type="fixed" name="camera_joint">
-      <origin xyz="0.092 0 0.05" rpy="-1.57 0 0" />
+      <origin xyz="0.2 0 0.05" rpy="0 1.57 0" />
       <child link="camera_link" />
       <parent link="base_link" />

Commit message: fix camera again.

File: mec_mobile_description/urdf/robots/robot_3d.urdf.xacro (robot description, xacro)
@@ -139,8 +139,7 @@
     <!-- 2.5.1 Camera physical properties -->
     <joint type="fixed" name="camera_joint">
-      <origin xyz="0.2 0 0.05" rpy="0 1.57 0" />
+      <origin xyz="0.2 0 0.15" rpy="0 1.5708 0" />
       <child link="camera_link" />
       <parent link="base_link" />
-      <axis xyz="0 1 0" />
     </joint>
     <link name='camera_link'>
@@ -165,12 +164,46 @@
     </link>
     <gazebo reference="camera_link">
-      <material>Gazebo/Red</material>
+      <sensor type="camera" name="camera_sensor_rig">
+        <update_rate>30.0</update_rate>
+        <visualize>true</visualize>
+        <camera name="camera">
+          <horizontal_fov>0.2</horizontal_fov>
+          <image>
+            <width>640</width>
+            <height>480</height>
+            <format>R8G8B8</format>
+          </image>
+          <clip>
+            <near>0.05</near>
+            <far>8.0</far>
+          </clip>
+        </camera>
+        <plugin name="camera_controller" filename="libgazebo_ros_camera.so">
+          <camera_name>camera</camera_name>
+          <frame_name>camera_link_optical</frame_name>
+          <ros>
+            <namespace>/camera</namespace>
+            <remapping>image_raw:=image_raw</remapping>
+            <remapping>camera_info:=camera_info</remapping>
+          </ros>
+        </plugin>
+      </sensor>
     </gazebo>
     <joint type="fixed" name="camera_optical_joint">
-      <origin xyz="0 0 0" rpy="-1.5707 0 -1.5707" />
+    <origin xyz="0 0 0" rpy="-1.5708 0 -1.5708" />
       <child link="camera_link_optical" />
       <parent link="camera_link" />
     </joint>
     <link name="camera_link_optical">
+      <inertial>
+        <mass value="0.0001" />
+        <origin xyz="0 0 0" rpy="0 0 0" />
+        <inertia ixx="1e-6" iyy="1e-6" izz="1e-6" ixy="0" ixz="0" iyz="0" />
+      </inertial>
+      <visual>
+        <geometry>
+          <box size="0.001 0.001 0.001" />
+        </geometry>
+      </visual>
     </link>
     <!-- 2.5.1 End -->
