Commit message: Kind of moves along line

File: arena-robot-simulation/mec_mobile_description/urdf/robots/robot_3d.urdf.xacro (robot description, xacro)
@@ -139,5 +139,5 @@
     <!-- 2.5.1 Camera physical properties -->
     <joint type="fixed" name="camera_joint">
-      <origin xyz="0.2 0 0.15" rpy="0 1.5708 0" />
+      <origin xyz="0.2 0 0.06" rpy="0 1.5708 0" />
       <child link="camera_link" />
       <parent link="base_link" />
