Commit message: add code

File: arena-robot-simulation/mec_mobile_description/urdf/sarm/sarm.urdf.xacro (robot description, xacro)
@@ -2,8 +2,5 @@
 <robot xmlns:xacro="http://www.ros.org/wiki/xacro" name="sarm">
   <xacro:property name="mass" value="1.0" />
-  <xacro:property
-        name="scale"
-        value="0.001"
-    />  <!-- Increased from 0.001 to 0.01 -->
+  <xacro:property name="scale" value="0.01" />
   <xacro:property name="inertia_val" value="0.01" />
   <link name="sarm_link">
@@ -12,13 +9,14 @@
       <geometry>
         <mesh
-                    filename="file://$(find mec_mobile_description)/meshes/sarm/sarm.stl"
+                    filename="file://$(find mec_mobile_description)/meshes/sarm/sarm.obj"
                     scale="${scale} ${scale} ${scale}"
                 />
       </geometry>
-      <material name="gray">
+      <!-- Remove or comment out the material section to use MTL materials -->
+      <!-- <material name="gray">
         <color rgba="0.7 0.7 0.7 1.0" />
-      </material>
+      </material> -->
     </visual>
-    <!-- Collision -->
+    <!-- Collision (keep STL for collision as it's more efficient) -->
     <collision>
       <geometry>

Commit message: spawn stl.

File: arena-robot-simulation/mec_mobile_description/urdf/sarm/sarm.urdf.xacro (robot description, xacro)
@@ -2,5 +2,5 @@
 <robot xmlns:xacro="http://www.ros.org/wiki/xacro" name="sarm">
   <xacro:property name="mass" value="1.0" />
-  <xacro:property name="scale" value="0.01" />
+  <xacro:property name="scale" value="0.001" />
   <xacro:property name="inertia_val" value="0.01" />
   <link name="sarm_link">
@@ -9,5 +9,5 @@
       <geometry>
         <mesh
-                    filename="file://$(find mec_mobile_description)/meshes/sarm/sarm.obj"
+                    filename="file://$(find mec_mobile_description)/meshes/sarm/sarm.stl"
                     scale="${scale} ${scale} ${scale}"
                 />

Commit message: add parameters to make collision physics workable. TODO: fix these parameters, TODO: separate links for each.

File: arena-robot-simulation/mec_mobile_description/urdf/sarm/sarm.urdf.xacro (robot description, xacro)
@@ -4,4 +4,24 @@
   <xacro:property name="scale" value="0.001" />
   <xacro:property name="inertia_val" value="0.01" />
+  <xacro:property name="total_width" value="${0.19940 * scale}" />
+  <xacro:property name="wheel_width" value="${0.0304 * scale}" />
+  <xacro:property name="wheel_radius" value="${0.0325 * scale}" />
+  <xacro:property name="total_height" value="${0.16225 * scale}" />
+  <xacro:property name="base_length" value="${0.300 * scale}" />
+  <xacro:property name="centered_length" value="${0.238 * scale}" />
+  <xacro:property
+        name="base_x_offset"
+        value="${(centered_length - base_length) / 2}"
+    />
+  <xacro:property name="base_size_x" value="${base_length}" />
+  <xacro:property
+        name="base_size_y"
+        value="${total_width - (2 * wheel_width)}"
+    />
+  <xacro:property
+        name="base_size_z"
+        value="${total_height - (2 * wheel_radius)}"
+    />
+  <xacro:property name="base_mass" value="${4.6 * scale * scale * scale}" />
   <link name="sarm_link">
     <!-- Visual -->
@@ -9,5 +29,5 @@
       <geometry>
         <mesh
-                    filename="file://$(find mec_mobile_description)/meshes/sarm/chassis.stl"
+                    filename="file://$(find mec_mobile_description)/meshes/sarm/sarm.obj"
                     scale="${scale} ${scale} ${scale}"
                 />
@@ -21,8 +41,5 @@
     <collision>
       <geometry>
-        <mesh
-                    filename="file://$(find mec_mobile_description)/meshes/sarm/chassis.stl"
-                    scale="${scale} ${scale} ${scale}"
-                />
+        <box size="${base_size_x} ${base_size_y} ${base_size_z}" />
       </geometry>
     </collision>

Commit message: add sarm_base and sarm

File: arena-robot-simulation/mec_mobile_description/urdf/sarm/sarm.urdf.xacro (robot description, xacro)
@@ -1,59 +1,100 @@
 <?xml version="1.0" ?>
-<robot xmlns:xacro="http://www.ros.org/wiki/xacro" name="sarm">
-  <xacro:property name="mass" value="1.0" />
-  <xacro:property name="scale" value="0.001" />
-  <xacro:property name="inertia_val" value="0.01" />
-  <xacro:property name="total_width" value="${0.19940 * scale}" />
-  <xacro:property name="wheel_width" value="${0.0304 * scale}" />
-  <xacro:property name="wheel_radius" value="${0.0325 * scale}" />
-  <xacro:property name="total_height" value="${0.16225 * scale}" />
-  <xacro:property name="base_length" value="${0.300 * scale}" />
-  <xacro:property name="centered_length" value="${0.238 * scale}" />
-  <xacro:property
-        name="base_x_offset"
-        value="${(centered_length - base_length) / 2}"
+<robot
+    name="robot_3d"
+    xmlns:xacro="http://www.ros.org/wiki/xacro"
+    xmlns:gz="http://gazebosim.org/schema"
+>
+    <xacro:property name="M_PI" value="3.1415926535897931" />
+    <xacro:arg name="robot_name" default="robot_3d" />
+    <xacro:arg name="prefix" default="" />
+    <xacro:arg name="use_gazebo" default="false" />
+    <xacro:include
+        filename="$(find mec_mobile_description)/urdf/mech/sarm_base.urdf.xacro"
     />
-  <xacro:property name="base_size_x" value="${base_length}" />
-  <xacro:property
-        name="base_size_y"
-        value="${total_width - (2 * wheel_width)}"
+    <xacro:include
+        filename="$(find sarm_base_control)/urdf/control/mec_mobile.gazebo"
     />
-  <xacro:property
-        name="base_size_z"
-        value="${total_height - (2 * wheel_radius)}"
+    <xacro:robot_3d_base prefix="$(arg prefix)" />
+    <xacro:mecanum_wheel
+        prefix="$(arg prefix)"
+        side="front_left"
+        x_reflect="1"
+        y_reflect="1"
     />
-  <xacro:property name="base_mass" value="${4.6 * scale * scale * scale}" />
-  <link name="sarm_link">
-    <!-- Visual -->
-    <visual>
-      <geometry>
-        <mesh
-                    filename="file://$(find mec_mobile_description)/meshes/sarm/chassis.stl"
-                    scale="${scale} ${scale} ${scale}"
-                />
-      </geometry>
-      <!-- Remove or comment out the material section to use MTL materials -->
-      <!-- <material name="gray">
-        <color rgba="0.7 0.7 0.7 1.0" />
-      </material> -->
-    </visual>
-    <!-- Collision (keep STL for collision as it's more efficient) -->
-    <collision>
-      <geometry>
-        <box size="${base_size_x} ${base_size_y} ${base_size_z}" />
-      </geometry>
-    </collision>
-    <!-- Inertial -->
-    <inertial>
-      <mass value="${mass}" />
-      <inertia
-                ixx="${inertia_val}"
-                ixy="0.0"
-                ixz="0.0"
-                iyy="${inertia_val}"
-                iyz="0.0"
-                izz="${inertia_val}"
-            />
-    </inertial>
-  </link>
+    <xacro:mecanum_wheel
+        prefix="$(arg prefix)"
+        side="front_right"
+        x_reflect="1"
+        y_reflect="-1"
+    />
+    <xacro:mecanum_wheel
+        prefix="$(arg prefix)"
+        side="back_left"
+        x_reflect="-1"
+        y_reflect="1"
+    />
+    <xacro:mecanum_wheel
+        prefix="$(arg prefix)"
+        side="back_right"
+        x_reflect="-1"
+        y_reflect="-1"
+    />
+    <!-- 2.4 add Gazebo frictions -->
+    <gazebo reference='front_left_wheel_link'>
+      <collision>
+        <surface>
+          <friction>
+            <ode>
+              <mu>1.5</mu>
+              <mu2>0.0</mu2>
+              <fdir1 gz:expressed_in="base_footprint">1 -1 0</fdir1>
+            </ode>
+          </friction>
+        </surface>
+      </collision>
+    </gazebo>
+    <gazebo reference='back_left_wheel_link'>
+      <collision>
+        <surface>
+          <friction>
+            <ode>
+              <mu>1.5</mu>
+              <mu2>0.0</mu2>
+              <fdir1 gz:expressed_in="base_footprint">1 1 0</fdir1>
+            </ode>
+          </friction>
+        </surface>
+      </collision>
+    </gazebo>
+    <gazebo reference='front_right_wheel_link'>
+      <collision>
+        <surface>
+          <friction>
+            <ode>
+              <mu>1.5</mu>
+              <mu2>0.0</mu2>
+              <fdir1 gz:expressed_in="base_footprint">1 1 0</fdir1>
+            </ode>
+          </friction>
+        </surface>
+      </collision>
+    </gazebo>
+    <gazebo reference='back_right_wheel_link'>
+      <collision>
+        <surface>
+          <friction>
+            <ode>
+              <mu>1.5</mu>
+              <mu2>0.0</mu2>
+              <fdir1 gz:expressed_in="base_footprint">1 -1 0</fdir1>
+            </ode>
+          </friction>
+        </surface>
+      </collision>
+    </gazebo>
+    <gazebo reference="base_link">
+      <mu1>0.000002</mu1>
+      <mu2>0.000002</mu2>
+      <!-- <material>Gazebo/Red</material> -->
+    </gazebo>
 </robot>

Commit message: fix xacro

File: arena-robot-simulation/mec_mobile_description/urdf/sarm/sarm.urdf.xacro (robot description, xacro)
@@ -1,67 +1,33 @@
 <?xml version="1.0" ?>
 <robot
-    name="robot_3d"
+    name="sarm"
     xmlns:xacro="http://www.ros.org/wiki/xacro"
     xmlns:gz="http://gazebosim.org/schema"
 >
     <xacro:property name="M_PI" value="3.1415926535897931" />
-    <xacro:arg name="robot_name" default="robot_3d" />
+    <xacro:arg name="robot_name" default="sarm" />
     <xacro:arg name="prefix" default="" />
     <xacro:arg name="use_gazebo" default="false" />
+    <!-- Include base and wheels -->
     <xacro:include
-        filename="$(find mec_mobile_description)/urdf/mech/sarm_base.urdf.xacro"
+        filename="$(find mec_mobile_description)/urdf/mech/robot_3d_base.urdf.xacro"
     />
-    <gazebo reference='front_left_wheel_link'>
-      <collision>
-        <surface>
-          <friction>
-            <ode>
-              <mu>1.5</mu>
-              <mu2>0.0</mu2>
-              <fdir1 gz:expressed_in="base_footprint">1 -1 0</fdir1>
-            </ode>
-          </friction>
-        </surface>
-      </collision>
-    </gazebo>
-    <gazebo reference='back_left_wheel_link'>
-      <collision>
-        <surface>
-          <friction>
-            <ode>
-              <mu>1.5</mu>
-              <mu2>0.0</mu2>
-              <fdir1 gz:expressed_in="base_footprint">1 1 0</fdir1>
-            </ode>
-          </friction>
-        </surface>
-      </collision>
-    </gazebo>
-    <gazebo reference='front_right_wheel_link'>
-      <collision>
-        <surface>
-          <friction>
-            <ode>
-              <mu>1.5</mu>
-              <mu2>0.0</mu2>
-              <fdir1 gz:expressed_in="base_footprint">1 1 0</fdir1>
-            </ode>
-          </friction>
-        </surface>
-      </collision>
-    </gazebo>
-    <gazebo reference='back_right_wheel_link'>
-      <collision>
-        <surface>
-          <friction>
-            <ode>
-              <mu>1.5</mu>
-              <mu2>0.0</mu2>
-              <fdir1 gz:expressed_in="base_footprint">1 -1 0</fdir1>
-            </ode>
-          </friction>
-        </surface>
-      </collision>
-    </gazebo>
+    <xacro:include
+        filename="$(find mec_mobile_description)/urdf/mech/sarm_mecanum_wheel.urdf.xacro"
+    />
+    <!-- Include sensors -->
+    <xacro:include
+        filename="$(find mec_mobile_description)/urdf/sensors/lidar.urdf.xacro"
+    />
+    <xacro:include
+        filename="$(find mec_mobile_description)/urdf/sensors/imu.urdf.xacro"
+    />
+    <!-- Include gazebo control -->
+    <xacro:include
+        filename="$(find mec_mobile_description)/urdf/control/mec_mobile.gazebo"
+    />
+    <!-- Instantiate robot base -->
+    <xacro:robot_3d_base prefix="$(arg prefix)" />
+    <!-- Wheels -->
     <xacro:sarm_mecanum_wheel
         prefix="$(arg prefix)"
@@ -88,3 +54,86 @@
         y_reflect="-1"
     />
+    <!-- Lidar -->
+    <xacro:lidar_sensor
+        prefix="$(arg prefix)"
+        parent="$(arg prefix)base_link"
+        frame_id="laser_frame"
+        xyz_offset="0 0 0.0825"
+        rpy_offset="0 0 ${M_PI}"
+        mesh_xyz_offset="0 0 0"
+        mesh_rpy_offset="${-M_PI/2} 0 0"
+        topic_name="scan"
+    />
+    <!-- IMU -->
+    <xacro:imu_sensor
+        prefix="$(arg prefix)"
+        parent="$(arg prefix)base_link"
+        frame_id="imu"
+        xyz_offset="0 0 0.006"
+        rpy_offset="0 0 0"
+        update_rate="15.0"
+        topic_name="imu/data"
+    />
+    <!-- Gazebo friction for wheels -->
+    <gazebo reference='$(arg prefix)front_left_wheel_link'>
+      <collision>
+        <surface>
+          <friction>
+            <ode>
+              <mu>1.5</mu>
+              <mu2>0.0</mu2>
+              <fdir1
+                            gz:expressed_in="$(arg prefix)base_footprint"
+                        >1 -1 0</fdir1>
+            </ode>
+          </friction>
+        </surface>
+      </collision>
+    </gazebo>
+    <gazebo reference='$(arg prefix)back_left_wheel_link'>
+      <collision>
+        <surface>
+          <friction>
+            <ode>
+              <mu>1.5</mu>
+              <mu2>0.0</mu2>
+              <fdir1 gz:expressed_in="$(arg prefix)base_footprint">1 1 0</fdir1>
+            </ode>
+          </friction>
+        </surface>
+      </collision>
+    </gazebo>
+    <gazebo reference='$(arg prefix)front_right_wheel_link'>
+      <collision>
+        <surface>
+          <friction>
+            <ode>
+              <mu>1.5</mu>
+              <mu2>0.0</mu2>
+              <fdir1 gz:expressed_in="$(arg prefix)base_footprint">1 1 0</fdir1>
+            </ode>
+          </friction>
+        </surface>
+      </collision>
+    </gazebo>
+    <gazebo reference='$(arg prefix)back_right_wheel_link'>
+      <collision>
+        <surface>
+          <friction>
+            <ode>
+              <mu>1.5</mu>
+              <mu2>0.0</mu2>
+              <fdir1
+                            gz:expressed_in="$(arg prefix)base_footprint"
+                        >1 -1 0</fdir1>
+            </ode>
+          </friction>
+        </surface>
+      </collision>
+    </gazebo>
+    <!-- Optional base friction -->
+    <gazebo reference="$(arg prefix)base_link">
+      <mu1>0.000002</mu1>
+      <mu2>0.000002</mu2>
+    </gazebo>
 </robot>
