Commit message: fix urdf

File: arena-robot-simulation/mec_mobile_description/urdf/mech/mecanum_wheel.urdf.xacro (robot description, xacro)
@@ -1,3 +1,3 @@
-<?xml version="1.0"?>
+<?xml version="1.0" ?>
 <robot xmlns:xacro="http://www.ros.org/wiki/xacro">
   <xacro:property name="wheel_radius" value="0.0325" />
@@ -10,32 +10,41 @@
     <link name="${prefix}${side}_wheel_link">
       <visual>
-        <origin xyz="0 0 0" rpy="${pi/2} 0 0"/>
+        <origin xyz="0 0 0" rpy="${pi/2} 0 0" />
         <geometry>
-          <mesh filename="file://$(find mec_mobile_description)/meshes/robot_3d/visual/${side}_wheel_X3.STL"/>
+          <mesh
+                        filename="file://$(find mec_mobile_description)/meshes/robot_3d/visual/${side}_wheel_X3.stl"
+                    />
         </geometry>
         <material name="dark_gray">
-          <color rgba="0.2 0.2 0.2 1.0"/>
+          <color rgba="0.2 0.2 0.2 1.0" />
         </material>
       </visual>
       <collision>
-        <origin xyz="0 0 0" rpy="${pi/2} 0 0"/>
+        <origin xyz="0 0 0" rpy="${pi/2} 0 0" />
         <geometry>
-          <cylinder radius="${wheel_radius}" length="${wheel_width}"/>
+          <cylinder radius="${wheel_radius}" length="${wheel_width}" />
         </geometry>
       </collision>
       <inertial>
-        <origin xyz="0 0 0" rpy="0 0 0"/>
-        <mass value="${wheel_mass}"/>
+        <origin xyz="0 0 0" rpy="0 0 0" />
+        <mass value="${wheel_mass}" />
         <inertia
-          ixx="${(wheel_mass/12.0) * (3*wheel_radius*wheel_radius + wheel_width*wheel_width)}" ixy="0" ixz="0"
-          iyy="${(wheel_mass/2.0) * (wheel_radius*wheel_radius)}" iyz="0"
-          izz="${(wheel_mass/12.0) * (3*wheel_radius*wheel_radius + wheel_width*wheel_width)}"/>
+                    ixx="${(wheel_mass/12.0) * (3*wheel_radius*wheel_radius + wheel_width*wheel_width)}"
+                    ixy="0"
+                    ixz="0"
+                    iyy="${(wheel_mass/2.0) * (wheel_radius*wheel_radius)}"
+                    iyz="0"
+                    izz="${(wheel_mass/12.0) * (3*wheel_radius*wheel_radius + wheel_width*wheel_width)}"
+                />
       </inertial>
     </link>
     <joint name="${prefix}${side}_wheel_joint" type="continuous">
-      <axis xyz="0 1 0"/>
-      <parent link="${prefix}base_link"/>
-      <child link="${prefix}${side}_wheel_link"/>
-      <origin xyz="${x_reflect*wheel_xoff} ${y_reflect*(wheel_separation/2+wheel_yoff)} ${-wheel_radius}" rpy="0 0 0"/>
+      <axis xyz="0 1 0" />
+      <parent link="${prefix}base_link" />
+      <child link="${prefix}${side}_wheel_link" />
+      <origin
+                xyz="${x_reflect*wheel_xoff} ${y_reflect*(wheel_separation/2+wheel_yoff)} ${-wheel_radius}"
+                rpy="0 0 0"
+            />
     </joint>
     <gazebo reference="${prefix}${side}_wheel_link">

File: arena-robot-simulation/mec_mobile_description/urdf/mech/robot_3d_base.urdf.xacro (robot description, xacro)
@@ -1,3 +1,3 @@
-<?xml version="1.0"?>
+<?xml version="1.0" ?>
 <robot xmlns:xacro="http://www.ros.org/wiki/xacro">
 <xacro:property name="scale" value="2.0" />  <!-- or any factor you want -->
@@ -8,35 +8,53 @@
 <xacro:property name="base_length" value="${0.300 * scale}" />
 <xacro:property name="centered_length" value="${0.238 * scale}" />
-<xacro:property name="base_x_offset" value="${(centered_length - base_length) / 2}" />
+<xacro:property
+        name="base_x_offset"
+        value="${(centered_length - base_length) / 2}"
+    />
 <xacro:property name="base_size_x" value="${base_length}" />
 <xacro:property name="base_size_y" value="${total_width - (2 * wheel_width)}" />
-<xacro:property name="base_size_z" value="${total_height - (2 * wheel_radius)}" />
+<xacro:property
+        name="base_size_z"
+        value="${total_height - (2 * wheel_radius)}"
+    />
 <xacro:property name="base_mass" value="${4.6 * scale * scale * scale}" />
 <xacro:macro name="robot_3d_base" params="prefix">
-  <link name="${prefix}base_footprint"/>
+  <link name="${prefix}base_footprint" />
   <link name="${prefix}base_link">
     <visual>
         <geometry>
-            <mesh filename="file://$(find mec_mobile_description)/meshes/robot_3d/visual/base_link_X3.STL"/>
+            <mesh
+                        filename="file://$(find mec_mobile_description)/meshes/robot_3d/visual/base_link_X3.stl"
+                    />
             <scale>${scale} ${scale} ${scale}</scale>
         </geometry>
         <material name="white">
-          <color rgba="1 1 1 1"/>
+          <color rgba="1 1 1 1" />
         </material>
-        <origin xyz="0 0 0" rpy="0 0 0"/>
+        <origin xyz="0 0 0" rpy="0 0 0" />
     </visual>
     <collision>
         <geometry>
-            <box size="${base_size_x} ${base_size_y} ${base_size_z}"/>
+            <box size="${base_size_x} ${base_size_y} ${base_size_z}" />
         </geometry>
-        <origin xyz="${base_x_offset} 0 ${base_size_z/2 + wheel_radius/4}" rpy="0 0 0"/>
+        <origin
+                    xyz="${base_x_offset} 0 ${base_size_z/2 + wheel_radius/4}"
+                    rpy="0 0 0"
+                />
     </collision>
     <inertial>
-        <origin xyz="${base_x_offset} 0 ${base_size_z/2 + wheel_radius/4}" rpy="0 0 0"/>
-        <mass value="${base_mass}"/>
+        <origin
+                    xyz="${base_x_offset} 0 ${base_size_z/2 + wheel_radius/4}"
+                    rpy="0 0 0"
+                />
+        <mass value="${base_mass}" />
         <inertia
-            ixx="${(1/12) * base_mass * ((base_size_y * base_size_y) + (base_size_z * base_size_z))}" ixy="0.0" ixz="0.0"
-            iyy="${(1/12) * base_mass * ((base_size_x * base_size_x) + (base_size_z * base_size_z))}" iyz="0.0"
-            izz="${(1/12) * base_mass * ((base_size_x * base_size_x) + (base_size_y * base_size_y))}"/>
+                    ixx="${(1/12) * base_mass * ((base_size_y * base_size_y) + (base_size_z * base_size_z))}"
+                    ixy="0.0"
+                    ixz="0.0"
+                    iyy="${(1/12) * base_mass * ((base_size_x * base_size_x) + (base_size_z * base_size_z))}"
+                    iyz="0.0"
+                    izz="${(1/12) * base_mass * ((base_size_x * base_size_x) + (base_size_y * base_size_y))}"
+                />
     </inertial>
   </link>
@@ -51,7 +69,7 @@
   </gazebo>
   <joint name="${prefix}base_joint" type="fixed">
-    <parent link="${prefix}base_footprint"/>
-    <child link="${prefix}base_link"/>
-    <origin xyz="0 0 ${wheel_radius}" rpy="0 0 0"/>
+    <parent link="${prefix}base_footprint" />
+    <child link="${prefix}base_link" />
+    <origin xyz="0 0 ${wheel_radius}" rpy="0 0 0" />
   </joint>
 </xacro:macro>

File: arena-robot-simulation/mec_mobile_description/urdf/mech/sarm_base.urdf.xacro (robot description, xacro)
@@ -93,5 +93,5 @@
         <geometry>
           <mesh
-                        filename="file://$(find mec_mobile_description)/meshes/sarm/visual/${side}_wheel.STL"
+                        filename="/home/ash-blake/lfr_ws/src/arena-robot-simulation/mec_mobile_description/meshes/sarm/visual/${side}_wheel.stl"
                     />
         </geometry>

File: arena-robot-simulation/mec_mobile_description/urdf/mech/sarm_mecanum_wheel.urdf.xacro (robot description, xacro)
@@ -16,5 +16,5 @@
         <geometry>
           <mesh
-                        filename="file://$(find mec_mobile_description)/meshes/sarm/visual/${side}_wheel.STL"
+                        filename="file://$(find mec_mobile_description)/meshes/sarm/visual/${side}_wheel.stl"
                     />
         </geometry>
