Commit message: TODO: fix xacro

File: arena-robot-simulation/mec_mobile_description/urdf/mech/sarm_base.urdf.xacro (robot description, xacro)
@@ -80,5 +80,67 @@
     </joint>
   </xacro:macro>
-  <!-- Instantiate SARM base -->
   <xacro:sarm_base prefix="sarm_" />
+  <xacro:macro
+        name="sarm_mecanum_wheel"
+        params="prefix side x_reflect y_reflect"
+    >
+    <link name="${prefix}${side}_wheel_link">
+      <visual>
+        <origin xyz="0 0 0" rpy="${pi/2} 0 0" />
+        <geometry>
+          <mesh
+                        filename="file://$(find mec_mobile_description)/meshes/sarm/visual/${side}_wheel.STL"
+                    />
+        </geometry>
+        <material name="dark_gray">
+          <color rgba="0.2 0.2 0.2 1.0" />
+        </material>
+      </visual>
+      <collision>
+        <origin xyz="0 0 0" rpy="${pi/2} 0 0" />
+        <geometry>
+          <cylinder radius="${wheel_radius}" length="${wheel_width}" />
+        </geometry>
+      </collision>
+      <inertial>
+        <origin xyz="0 0 0" rpy="0 0 0" />
+        <mass value="${wheel_mass}" />
+        <inertia
+                    ixx="${(wheel_mass/12.0) * (3*wheel_radius*wheel_radius + wheel_width*wheel_width)}"
+                    ixy="0"
+                    ixz="0"
+                    iyy="${(wheel_mass/2.0) * (wheel_radius*wheel_radius)}"
+                    iyz="0"
+                    izz="${(wheel_mass/12.0) * (3*wheel_radius*wheel_radius + wheel_width*wheel_width)}"
+                />
+      </inertial>
+    </link>
+    <joint name="${prefix}${side}_wheel_joint" type="continuous">
+      <axis xyz="0 1 0" />
+      <parent link="${prefix}base_link" />
+      <child link="${prefix}${side}_wheel_link" />
+      <origin
+                xyz="${x_reflect*wheel_xoff} ${y_reflect*(wheel_separation/2+wheel_yoff)} ${-wheel_radius}"
+                rpy="0 0 0"
+            />
+    </joint>
+    <gazebo reference="${prefix}${side}_wheel_link">
+      <surface>
+        <friction>
+          <ode>
+              <mu>1.0</mu>
+              <mu2>0.0</mu2>
+          </ode>
+        </friction>
+      </surface>
+      <visual>
+          <material>
+              <ambient>0.2 0.2 0.2 1.0</ambient>
+              <diffuse>0.2 0.2 0.2 1.0</diffuse>
+              <specular>0.2 0.2 0.2 1.0</specular>
+              <emissive>0.0 0.0 0.0 0.0</emissive>
+          </material>
+      </visual>
+  </gazebo>
+  </xacro:macro>
 </robot>

File: arena-robot-simulation/mec_mobile_description/urdf/robots/robot_3d.urdf.xacro (robot description, xacro)
@@ -79,5 +79,4 @@
         topic_name="imu/data"
     />
-    <!-- 2.4 add Gazebo frictions -->
     <gazebo reference='front_left_wheel_link'>
       <collision>

File: arena-robot-simulation/mec_mobile_description/urdf/sarm/sarm.urdf.xacro (robot description, xacro)
@@ -12,33 +12,4 @@
         filename="$(find mec_mobile_description)/urdf/mech/sarm_base.urdf.xacro"
     />
-    <xacro:include
-        filename="$(find sarm_base_control)/urdf/control/mec_mobile.gazebo"
-    />
-    <xacro:robot_3d_base prefix="$(arg prefix)" />
-    <xacro:mecanum_wheel
-        prefix="$(arg prefix)"
-        side="front_left"
-        x_reflect="1"
-        y_reflect="1"
-    />
-    <xacro:mecanum_wheel
-        prefix="$(arg prefix)"
-        side="front_right"
-        x_reflect="1"
-        y_reflect="-1"
-    />
-    <xacro:mecanum_wheel
-        prefix="$(arg prefix)"
-        side="back_left"
-        x_reflect="-1"
-        y_reflect="1"
-    />
-    <xacro:mecanum_wheel
-        prefix="$(arg prefix)"
-        side="back_right"
-        x_reflect="-1"
-        y_reflect="-1"
-    />
-    <!-- 2.4 add Gazebo frictions -->
     <gazebo reference='front_left_wheel_link'>
       <collision>
@@ -93,8 +64,27 @@
       </collision>
     </gazebo>
-    <gazebo reference="base_link">
-      <mu1>0.000002</mu1>
-      <mu2>0.000002</mu2>
-      <!-- <material>Gazebo/Red</material> -->
-    </gazebo>
+    <xacro:sarm_mecanum_wheel
+        prefix="$(arg prefix)"
+        side="front_left"
+        x_reflect="1"
+        y_reflect="1"
+    />
+    <xacro:sarm_mecanum_wheel
+        prefix="$(arg prefix)"
+        side="front_right"
+        x_reflect="1"
+        y_reflect="-1"
+    />
+    <xacro:sarm_mecanum_wheel
+        prefix="$(arg prefix)"
+        side="back_left"
+        x_reflect="-1"
+        y_reflect="1"
+    />
+    <xacro:sarm_mecanum_wheel
+        prefix="$(arg prefix)"
+        side="back_right"
+        x_reflect="-1"
+        y_reflect="-1"
+    />
 </robot>

Commit message: TODO: fix missing launch_description

File: arena-robot-simulation/mec_mobile_description/urdf/mech/sarm_base.urdf.xacro (robot description, xacro)
@@ -20,4 +20,7 @@
     />
   <xacro:property name="base_mass" value="${4.6 * scale * scale * scale}" />
+  <xacro:property name="wheel_xoff" value="0.05" />
+  <xacro:property name="wheel_yoff" value="0.0" />
+  <xacro:property name="wheel_separation" value="0.15" />
   <!-- Macro -->
   <xacro:macro name="sarm_base" params="prefix">
@@ -103,16 +106,4 @@
         </geometry>
       </collision>
-      <inertial>
-        <origin xyz="0 0 0" rpy="0 0 0" />
-        <mass value="${wheel_mass}" />
-        <inertia
-                    ixx="${(wheel_mass/12.0) * (3*wheel_radius*wheel_radius + wheel_width*wheel_width)}"
-                    ixy="0"
-                    ixz="0"
-                    iyy="${(wheel_mass/2.0) * (wheel_radius*wheel_radius)}"
-                    iyz="0"
-                    izz="${(wheel_mass/12.0) * (3*wheel_radius*wheel_radius + wheel_width*wheel_width)}"
-                />
-      </inertial>
     </link>
     <joint name="${prefix}${side}_wheel_joint" type="continuous">

Commit message: everything imports, but dimensions messed up. TODO: dimensions fix.

File: arena-robot-simulation/mec_mobile_description/urdf/mech/sarm_base.urdf.xacro (robot description, xacro)
@@ -1,4 +1,4 @@
 <?xml version="1.0" ?>
-<robot xmlns:xacro="http://www.ros.org/wiki/xacro" name="sarm">
+<robot xmlns:xacro="http://www.ros.org/wiki/xacro">
   <!-- Properties -->
   <xacro:property name="scale" value="0.001" />
@@ -82,55 +82,3 @@
     </joint>
   </xacro:macro>
-  <xacro:sarm_base prefix="sarm_" />
-  <xacro:macro
-        name="sarm_mecanum_wheel"
-        params="prefix side x_reflect y_reflect"
-    >
-    <link name="${prefix}${side}_wheel_link">
-      <visual>
-        <origin xyz="0 0 0" rpy="${pi/2} 0 0" />
-        <geometry>
-          <mesh
-                        filename="/home/hephan/lfr_ws/src/arena-robot-simulation/mec_mobile_description/meshes/sarm/visual/${side}_wheel.stl"
-                    />
-        </geometry>
-        <material name="dark_gray">
-          <color rgba="0.2 0.2 0.2 1.0" />
-        </material>
-      </visual>
-      <collision>
-        <origin xyz="0 0 0" rpy="${pi/2} 0 0" />
-        <geometry>
-          <cylinder radius="${wheel_radius}" length="${wheel_width}" />
-        </geometry>
-      </collision>
-    </link>
-    <joint name="${prefix}${side}_wheel_joint" type="continuous">
-      <axis xyz="0 1 0" />
-      <parent link="${prefix}base_link" />
-      <child link="${prefix}${side}_wheel_link" />
-      <origin
-                xyz="${x_reflect*wheel_xoff} ${y_reflect*(wheel_separation/2+wheel_yoff)} ${-wheel_radius}"
-                rpy="0 0 0"
-            />
-    </joint>
-    <gazebo reference="${prefix}${side}_wheel_link">
-      <surface>
-        <friction>
-          <ode>
-              <mu>1.0</mu>
-              <mu2>0.0</mu2>
-          </ode>
-        </friction>
-      </surface>
-      <visual>
-          <material>
-              <ambient>0.2 0.2 0.2 1.0</ambient>
-              <diffuse>0.2 0.2 0.2 1.0</diffuse>
-              <specular>0.2 0.2 0.2 1.0</specular>
-              <emissive>0.0 0.0 0.0 0.0</emissive>
-          </material>
-      </visual>
-  </gazebo>
-  </xacro:macro>
 </robot>

File: arena-robot-simulation/mec_mobile_description/urdf/mech/sarm_mecanum_wheel.urdf.xacro (robot description, xacro)
@@ -1,10 +1,14 @@
 <?xml version="1.0" ?>
 <robot xmlns:xacro="http://www.ros.org/wiki/xacro">
-  <xacro:property name="wheel_radius" value="0.0325" />
-  <xacro:property name="wheel_separation" value="0.169" />
-  <xacro:property name="wheel_width" value="0.03040" />
-  <xacro:property name="wheel_mass" value="9.1" />
-  <xacro:property name="wheel_xoff" value="0.08" />
-  <xacro:property name="wheel_yoff" value="-0.01" />
+<xacro:property name="scale" value="0.001" />
+  <xacro:property
+        name="wheel_radius"
+        value="${0.0325 * scale}"
+    /> <!-- Remove hardcoded values -->
+  <xacro:property name="wheel_separation" value="${0.169}" />
+  <xacro:property name="wheel_width" value="${0.03040 * scale}" />
+  <xacro:property name="wheel_mass" value="${9.1 * scale * scale * scale}" />
+  <xacro:property name="wheel_xoff" value="${0.08}" />
+  <xacro:property name="wheel_yoff" value="${-0.01}" />
   <xacro:macro
         name="sarm_mecanum_wheel"

File: arena-robot-simulation/mec_mobile_description/urdf/sarm/sarm.urdf.xacro (robot description, xacro)
@@ -7,9 +7,9 @@
     <xacro:property name="M_PI" value="3.1415926535897931" />
     <xacro:arg name="robot_name" default="sarm" />
-    <xacro:arg name="prefix" default="" />
+    <xacro:arg name="prefix" default="sarm_" />
     <xacro:arg name="use_gazebo" default="false" />
     <!-- Include base and wheels -->
     <xacro:include
-        filename="$(find mec_mobile_description)/urdf/mech/robot_3d_base.urdf.xacro"
+        filename="$(find mec_mobile_description)/urdf/mech/sarm_base.urdf.xacro"
     />
     <xacro:include
@@ -17,10 +17,10 @@
     />
     <!-- Include sensors -->
-    <xacro:include
+    <!-- <xacro:include
         filename="$(find mec_mobile_description)/urdf/sensors/lidar.urdf.xacro"
     />
     <xacro:include
         filename="$(find mec_mobile_description)/urdf/sensors/imu.urdf.xacro"
-    />
+    /> -->
     <!-- Include gazebo control -->
     <!-- <xacro:include
@@ -28,5 +28,5 @@
     /> -->
     <!-- Instantiate robot base -->
-    <xacro:robot_3d_base prefix="$(arg prefix)" />
+    <xacro:sarm_base prefix="$(arg prefix)" />
     <!-- Wheels -->
     <xacro:sarm_mecanum_wheel

Commit message: fix scaling

File: arena-robot-simulation/mec_mobile_description/urdf/mech/sarm_base.urdf.xacro (robot description, xacro)
@@ -2,11 +2,11 @@
 <robot xmlns:xacro="http://www.ros.org/wiki/xacro">
   <!-- Properties -->
-  <xacro:property name="scale" value="0.001" />
-  <xacro:property name="wheel_radius" value="${0.0325 * scale}" />
-  <xacro:property name="wheel_width" value="${0.0304 * scale}" />
-  <xacro:property name="total_width" value="${0.1994 * scale}" />
-  <xacro:property name="total_height" value="${0.16225 * scale}" />
-  <xacro:property name="base_length" value="${0.3 * scale}" />
-  <xacro:property name="centered_length" value="${0.238 * scale}" />
+  <xacro:property name="scale" value="0.0001" />
+  <xacro:property name="wheel_radius" value="${35 * scale}" />
+  <xacro:property name="wheel_width" value="${30.5 * scale}" />
+  <xacro:property name="total_width" value="${360 * scale}" />
+  <xacro:property name="total_height" value="${140 * scale}" />
+  <xacro:property name="base_length" value="${300 * scale}" />
+  <xacro:property name="centered_length" value="${38.5 * scale}" />
   <xacro:property
         name="base_x_offset"
@@ -33,4 +33,5 @@
           <mesh
                         filename="file://$(find mec_mobile_description)/meshes/sarm/chassis.stl"
+                        scale="${scale} ${scale} ${scale}"
                     />
         </geometry>

File: arena-robot-simulation/mec_mobile_description/urdf/mech/sarm_mecanum_wheel.urdf.xacro (robot description, xacro)
@@ -9,6 +9,6 @@
   <xacro:property name="wheel_width" value="${0.03040 * scale}" />
   <xacro:property name="wheel_mass" value="${9.1 * scale * scale * scale}" />
-  <xacro:property name="wheel_xoff" value="${0.08}" />
-  <xacro:property name="wheel_yoff" value="${-0.01}" />
+  <xacro:property name="wheel_xoff" value="${0.02}" />
+  <xacro:property name="wheel_yoff" value="${0}" />
   <xacro:macro
         name="sarm_mecanum_wheel"
@@ -17,5 +17,5 @@
     <link name="${prefix}${side}_wheel_link">
       <visual>
-        <origin xyz="0 0 0" rpy="${pi/2} 0 0" />
+        <origin xyz="0 0 0" rpy="0 0 0" />
         <geometry>
           <mesh
@@ -52,5 +52,5 @@
       <child link="${prefix}${side}_wheel_link" />
       <origin
-                xyz="${x_reflect*wheel_xoff} ${y_reflect*(wheel_separation/2+wheel_yoff)} ${-wheel_radius}"
+                xyz="${x_reflect*wheel_xoff} ${y_reflect*(wheel_separation/2+wheel_yoff)} 0"
                 rpy="0 0 0"
             />

Commit message: fix values.

File: arena-robot-simulation/mec_mobile_description/urdf/mech/sarm_base.urdf.xacro (robot description, xacro)
@@ -2,5 +2,5 @@
 <robot xmlns:xacro="http://www.ros.org/wiki/xacro">
   <!-- Properties -->
-  <xacro:property name="scale" value="0.0001" />
+  <xacro:property name="scale" value="0.001" />
   <xacro:property name="wheel_radius" value="${35 * scale}" />
   <xacro:property name="wheel_width" value="${30.5 * scale}" />
@@ -22,5 +22,5 @@
   <xacro:property name="wheel_xoff" value="0.05" />
   <xacro:property name="wheel_yoff" value="0.0" />
-  <xacro:property name="wheel_separation" value="0.15" />
+  <xacro:property name="wheel_separation" value="0.169" />
   <!-- Macro -->
   <xacro:macro name="sarm_base" params="prefix">

File: arena-robot-simulation/mec_mobile_description/urdf/mech/sarm_mecanum_wheel.urdf.xacro (robot description, xacro)
@@ -6,5 +6,5 @@
         value="${0.0325 * scale}"
     /> <!-- Remove hardcoded values -->
-  <xacro:property name="wheel_separation" value="${0.169}" />
+  <xacro:property name="wheel_separation" value="0.169" />
   <xacro:property name="wheel_width" value="${0.03040 * scale}" />
   <xacro:property name="wheel_mass" value="${9.1 * scale * scale * scale}" />

Commit message: fix some values.

File: arena-robot-simulation/mec_mobile_description/urdf/mech/sarm_base.urdf.xacro (robot description, xacro)
@@ -3,5 +3,5 @@
   <!-- Properties -->
   <xacro:property name="scale" value="0.001" />
-  <xacro:property name="wheel_radius" value="${35 * scale}" />
+  <xacro:property name="wheel_radius" value="${3.5 * scale}" />
   <xacro:property name="wheel_width" value="${30.5 * scale}" />
   <xacro:property name="total_width" value="${360 * scale}" />
@@ -20,5 +20,5 @@
     />
   <xacro:property name="base_mass" value="${4.6 * scale * scale * scale}" />
-  <xacro:property name="wheel_xoff" value="0.05" />
+  <xacro:property name="wheel_xoff" value="0.02" />
   <xacro:property name="wheel_yoff" value="0.0" />
   <xacro:property name="wheel_separation" value="0.169" />

File: arena-robot-simulation/mec_mobile_description/urdf/mech/sarm_mecanum_wheel.urdf.xacro (robot description, xacro)
@@ -4,11 +4,11 @@
   <xacro:property
         name="wheel_radius"
-        value="${0.0325 * scale}"
+        value="${3.5 * scale}"
     /> <!-- Remove hardcoded values -->
   <xacro:property name="wheel_separation" value="0.169" />
-  <xacro:property name="wheel_width" value="${0.03040 * scale}" />
+  <xacro:property name="wheel_width" value="${30.5 * scale}" />
   <xacro:property name="wheel_mass" value="${9.1 * scale * scale * scale}" />
-  <xacro:property name="wheel_xoff" value="${0.02}" />
-  <xacro:property name="wheel_yoff" value="${0}" />
+  <xacro:property name="wheel_xoff" value="0.02" />
+  <xacro:property name="wheel_yoff" value="0" />
   <xacro:macro
         name="sarm_mecanum_wheel"
@@ -21,5 +21,5 @@
           <mesh
                         filename="file://$(find mec_mobile_description)/meshes/sarm/visual/${side}_wheel.stl"
-                        scale="0.001 0.001 0.001"
+                        scale="${scale} ${scale} ${scale}"
                     />
         </geometry>
@@ -52,5 +52,5 @@
       <child link="${prefix}${side}_wheel_link" />
       <origin
-                xyz="${x_reflect*wheel_xoff} ${y_reflect*(wheel_separation/2+wheel_yoff)} 0"
+                xyz="${x_reflect*wheel_xoff} ${y_reflect*(wheel_separation/2+wheel_yoff)} -${wheel_radius}"
                 rpy="0 0 0"
             />

File: arena-robot-simulation/mec_mobile_description/urdf/sarm/sarm.urdf.xacro (robot description, xacro)
@@ -40,5 +40,5 @@
         side="front_right"
         x_reflect="1"
-        y_reflect="-1"
+        y_reflect="1"
     />
     <xacro:sarm_mecanum_wheel
@@ -52,5 +52,5 @@
         side="back_right"
         x_reflect="-1"
-        y_reflect="-1"
+        y_reflect="1"
     />
     <!-- Gazebo friction for wheels -->

Commit message: fix sarm.

File: arena-robot-simulation/mec_mobile_description/urdf/mech/sarm_base.urdf.xacro (robot description, xacro)
@@ -22,5 +22,5 @@
   <xacro:property name="wheel_xoff" value="0.02" />
   <xacro:property name="wheel_yoff" value="0.0" />
-  <xacro:property name="wheel_separation" value="0.169" />
+  <xacro:property name="wheel_separation" value="${0.169 * scale}" />
   <!-- Macro -->
   <xacro:macro name="sarm_base" params="prefix">

File: arena-robot-simulation/mec_mobile_description/urdf/mech/sarm_mecanum_wheel.urdf.xacro (robot description, xacro)
@@ -6,5 +6,5 @@
         value="${3.5 * scale}"
     /> <!-- Remove hardcoded values -->
-  <xacro:property name="wheel_separation" value="0.169" />
+  <xacro:property name="wheel_separation" value="${0.169 * scale}" />
   <xacro:property name="wheel_width" value="${30.5 * scale}" />
   <xacro:property name="wheel_mass" value="${9.1 * scale * scale * scale}" />

Commit message: fix. TODO: programming.

File: arena-robot-simulation/mec_mobile_description/urdf/mech/sarm_base.urdf.xacro (robot description, xacro)
@@ -6,6 +6,6 @@
   <xacro:property name="wheel_width" value="${30.5 * scale}" />
   <xacro:property name="total_width" value="${360 * scale}" />
-  <xacro:property name="total_height" value="${140 * scale}" />
-  <xacro:property name="base_length" value="${300 * scale}" />
+  <xacro:property name="total_height" value="${100 * scale}" />
+  <xacro:property name="base_length" value="${225 * scale}" />
   <xacro:property name="centered_length" value="${38.5 * scale}" />
   <xacro:property
